File: pcb/555-gitaar-pedal/555-gitaar-pedal.kicad_sch (KiCad schematic)
At the start: 9 parts, among them Q1 BC547, U1 NE555P, U2 LM386

Commit message: plaatje
Parts:
- added C4: 220uF, symbol Device:C_Polarized_Small_US
- added J1: Geluid_UIT, symbol Connector_Audio:AudioPlug2
- added R3: 470, symbol Device:R_Small_US
- added RV2: 100k, symbol Device:R_Potentiometer_Small
- C2: value C_Small -> 1uF
Connections:
- net +9V: now also R3.1, R3.2
- net GND: now also U1.1 (GND), C4.2, J1.S
- net TRIG: now reaches U1.2 (TR)
- net TRIG: now also U1.6 (THR), C4.1, RV2.3
- net at U1.7 (DIS): now also RV2.2
- net at C3.2: now also J1.T
- no-connect marks 0 -> 2
Other:
- note added: "OUT"
- moved on the sheet: C1, C2, C3, RV1, U2

Commit message: KiCAD schema bijgewerkt
Other:
- company: (none) -> door Michiel Erasmus
- title: (none) -> 555-gitaar pedal
Changed lines of the file:
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@@
 (kicad_sch (version 20230121) (generator eeschema)
   (paper "A4")
+  (title_block
+    (title "555-gitaar pedal")
+    (date "2023-09-20")
+    (company "door Michiel Erasmus")
+    (comment 1 "michiel@voorspoed.ru")
+    (comment 2 "Easylab4kids")
+  )
   (junction (at 90.805 57.658) (diameter 0) (color 0 0 0 0)
   )

Commit message: KiCAD schema bijgewerkt
Parts:
- added D1: Tap, symbol Device:LED_Small
Connections:
- net GND: now also D1.1 (K)
- net at R1.1, U1.3 (Q): now also D1.2 (A)
- no-connect marks 2 -> 3
Other:
- moved on the sheet: R1
Changed lines of the file:
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@@
     (comment 2 "Easylab4kids")
+  )
+  (junction (at 118.618 71.501) (diameter 0) (color 0 0 0 0)
   )
   (junction (at 90.805 57.658) (diameter 0) (color 0 0 0 0)
@@
   (no_connect (at 66.802 110.49))
   (no_connect (at 84.582 76.581))
+  (no_connect (at 82.55 62.611))
   (wire (pts (xy 77.089 57.658) (xy 77.089 81.661))
     (stroke (width 0) (type default))
@@
     (stroke (width 0) (type default))
   )
+  (wire (pts (xy 118.618 71.501) (xy 120.269 71.501))
+    (stroke (width 0) (type default))
+  )
   (wire (pts (xy 83.439 118.11) (xy 94.234 118.11))
     (stroke (width 0) (type default))
@@
     (stroke (width 0) (type default))
   )
+  (wire (pts (xy 118.618 78.74) (xy 118.618 79.629))
+    (stroke (width 0) (type default))
+  )
   (wire (pts (xy 82.55 71.501) (xy 84.582 71.501))
     (stroke (width 0) (type default))
@@
     (stroke (width 0) (type default))
   )
+  (wire (pts (xy 111.887 81.661) (xy 109.982 81.661))
+    (stroke (width 0) (type default))
+  )
   (wire (pts (xy 57.277 115.57) (xy 57.277 107.315))
     (stroke (width 0) (type default))
@@
     (stroke (width 0) (type default))
   )
+  (wire (pts (xy 125.349 71.501) (xy 126.746 71.501))
+    (stroke (width 0) (type default))
+  )
   (wire (pts (xy 97.282 57.658) (xy 90.805 57.658))
     (stroke (width 0) (type default))
@@
     (stroke (width 0) (type default))
   )
-  (wire (pts (xy 121.539 71.501) (xy 126.746 71.501))
-    (stroke (width 0) (type default))
-  )
   (wire (pts (xy 134.366 76.581) (xy 134.366 80.137))
     (stroke (width 0) (type default))
   )
+  (wire (pts (xy 118.618 71.501) (xy 118.618 73.66))
+    (stroke (width 0) (type default))
+  )
   (wire (pts (xy 69.342 125.73) (xy 69.342 127.508))
     (stroke (width 0) (type default))
   )
-  (wire (pts (xy 109.982 81.661) (xy 114.427 81.661))
-    (stroke (width 0) (type default))
-  )
   (wire (pts (xy 41.148 110.109) (xy 45.593 110.109))
     (stroke (width 0) (type default))
@@
     (stroke (width 0) (type default))
   )
-  (wire (pts (xy 109.982 71.501) (xy 116.459 71.501))
+  (wire (pts (xy 109.982 71.501) (xy 118.618 71.501))
     (stroke (width 0) (type default))
   )
@@
     )
   )
-  (global_label "TRIG" (shape output) (at 114.427 81.661 0) (fields_autoplaced)
+  (global_label "TRIG" (shape output) (at 111.887 81.661 0) (fields_autoplaced)
     (effects (font (size 0.7 0.7)) (justify left))
-    (property "Intersheetrefs" "${INTERSHEET_REFS}" (at 118.3389 81.661 0)
+    (property "Intersheetrefs" "${INTERSHEET_REFS}" (at 115.7989 81.661 0)
       (effects (font (size 1.27 1.27)) (justify left) hide)
     )
@@
     )
   )
-  (symbol (lib_id "Device:R_Small_US") (at 118.999 71.501 90) (unit 1)
-    (in_bom yes) (on_board yes) (dnp no)
-    (property "Reference" "R1" (at 118.872 68.326 90)
+  (symbol (lib_id "Device:LED_Small") (at 118.618 76.2 90) (unit 1)
+    (in_bom yes) (on_board yes) (dnp no) (fields_autoplaced)
+    (property "Reference" "D1" (at 120.65 75.5015 90)
+      (effects (font (size 0.8 0.8)) (justify right))
+    )
+    (property "Value" "Tap" (at 120.65 77.4065 90)
+      (effects (font (size 0.77 0.77)) (justify right))
+    )
+    (property "Footprint" "" (at 118.618 76.2 90)
+      (effects (font (size 1.27 1.27)) hide)
+    )
+    (property "Datasheet" "~" (at 118.618 76.2 90)
+      (effects (font (size 1.27 1.27)) hide)
+    )
+    (pin "1")
+    (pin "2")
+    (instances
+      (project "555-gitaar-pedal"
+        (path "/a176e3ad-e522-4300-abee-2d729589d26e"
+          (reference "D1") (unit 1)
+        )
+      )
+    )
+  )
+  (symbol (lib_id "Device:R_Small_US") (at 122.809 71.501 90) (unit 1)
+    (in_bom yes) (on_board yes) (dnp no)
+    (property "Reference" "R1" (at 122.682 68.326 90)
       (effects (font (size 1.27 1.27)))
     )
-    (property "Value" "470" (at 118.872 69.85 90)
+    (property "Value" "470" (at 122.682 69.85 90)
       (effects (font (size 0.77 0.77)))
     )
-    (property "Footprint" "" (at 118.999 71.501 0)
-      (effects (font (size 1.27 1.27)) hide)
-    )
-    (property "Datasheet" "~" (at 118.999 71.501 0)
+    (property "Footprint" "" (at 122.809 71.501 0)
+      (effects (font (size 1.27 1.27)) hide)
+    )
+    (property "Datasheet" "~" (at 122.809 71.501 0)
       (effects (font (size 1.27 1.27)) hide)
     )
@@
         )
       )
+    )
+  )
+  (symbol (lib_id "power:GND") (at 118.618 79.629 0) (unit 1)
+    (in_bom yes) (on_board yes) (dnp no)
+    (property "Reference" "#PWR06" (at 118.618 85.979 0)
+      (effects (font (size 1.27 1.27)) hide)
+    )
+    (property "Value" "GND" (at 118.618 83.185 0)
+      (effects (font (size 0.77 0.77)))
+    )
+    (property "Footprint" "" (at 118.618 79.629 0)
+      (effects (font (size 1.27 1.27)) hide)
+    )
+    (property "Datasheet" "" (at 118.618 79.629 0)
+      (effects (font (size 1.27 1.27)) hide)
+    )
+    (pin "1")
+    (instances
+      (project "555-gitaar-pedal"
+        (path "/a176e3ad-e522-4300-abee-2d729589d26e"
+          (reference "#PWR06") (unit 1)
+        )
+      )

Commit message: KiCAD schema bijgewerkt
Parts:
- C1, C2, C3, C4: footprint (none) -> Capacitor_THT:CP_Axial_L10.0mm_D6.0mm_P15.00mm_Horizontal
- D1: footprint (none) -> LED_THT:LED_D3.0mm
- R1, R2, R3, RV1, RV2: footprint (none) -> Resistor_THT:R_Axial_DIN0309_L9.0mm_D3.2mm_P5.08mm_Vertical
- U2: footprint (none) -> Package_DIP:DIP-8_W7.62mm_Socket
Changed lines of the file:
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@@
   (junction (at 118.618 71.501) (diameter 0) (color 0 0 0 0)
   )
+  (junction (at 97.282 93.091) (diameter 0) (color 0 0 0 0)
+  )
   (junction (at 90.805 57.658) (diameter 0) (color 0 0 0 0)
   )
   (junction (at 45.593 120.65) (diameter 0) (color 0 0 0 0)
   )
+  (junction (at 77.089 57.658) (diameter 0) (color 0 0 0 0)
+  )
+  (junction (at 82.55 71.501) (diameter 0) (color 0 0 0 0)
+  )
   (junction (at 64.262 128.778) (diameter 0) (color 0 0 0 0)
   )
-  (junction (at 77.089 57.658) (diameter 0) (color 0 0 0 0)
-  )
-  (junction (at 82.55 71.501) (diameter 0) (color 0 0 0 0)
-  )
   (junction (at 79.375 83.439) (diameter 0) (color 0 0 0 0)
   )
   (junction (at 55.372 120.65) (diameter 0) (color 0 0 0 0)
-  )
-  (junction (at 97.282 93.091) (diameter 0) (color 0 0 0 0)
   )
   (no_connect (at 66.802 110.49))
@@
     (stroke (width 0) (type default))
   )
+  (wire (pts (xy 79.375 83.439) (xy 79.375 85.852))
+    (stroke (width 0) (type default))
+  )
+  (wire (pts (xy 134.366 62.992) (xy 134.366 66.421))
+    (stroke (width 0) (type default))
+  )
+  (wire (pts (xy 79.375 71.501) (xy 82.55 71.501))
+    (stroke (width 0) (type default))
+  )
+  (wire (pts (xy 55.372 128.778) (xy 55.372 120.65))
+    (stroke (width 0) (type default))
+  )
+  (wire (pts (xy 59.182 115.57) (xy 57.277 115.57))
+    (stroke (width 0) (type default))
+  )
+  (wire (pts (xy 118.618 71.501) (xy 120.269 71.501))
+    (stroke (width 0) (type default))
+  )
+  (wire (pts (xy 83.439 118.11) (xy 94.234 118.11))
+    (stroke (width 0) (type default))
+  )
   (wire (pts (xy 64.262 107.188) (xy 64.262 110.49))
     (stroke (width 0) (type default))
   )
+  (wire (pts (xy 90.805 56.134) (xy 90.805 57.658))
+    (stroke (width 0) (type default))
+  )
+  (wire (pts (xy 64.262 128.778) (xy 64.262 136.271))
+    (stroke (width 0) (type default))
+  )
+  (wire (pts (xy 85.09 65.151) (xy 114.427 65.151))
+    (stroke (width 0) (type default))
+  )
+  (wire (pts (xy 49.657 107.315) (xy 48.133 107.315))
+    (stroke (width 0) (type default))
+  )
+  (wire (pts (xy 45.593 117.475) (xy 45.593 120.65))
+    (stroke (width 0) (type default))
+  )
   (wire (pts (xy 97.282 86.741) (xy 97.282 93.091))
     (stroke (width 0) (type default))
   )
-  (wire (pts (xy 79.375 83.439) (xy 79.375 85.852))
-    (stroke (width 0) (type default))
-  )
-  (wire (pts (xy 134.366 62.992) (xy 134.366 66.421))
-    (stroke (width 0) (type default))
-  )
-  (wire (pts (xy 79.375 71.501) (xy 82.55 71.501))
-    (stroke (width 0) (type default))
-  )
-  (wire (pts (xy 55.372 128.778) (xy 55.372 120.65))
-    (stroke (width 0) (type default))
-  )
-  (wire (pts (xy 59.182 115.57) (xy 57.277 115.57))
-    (stroke (width 0) (type default))
-  )
-  (wire (pts (xy 118.618 71.501) (xy 120.269 71.501))
-    (stroke (width 0) (type default))
-  )
-  (wire (pts (xy 83.439 118.11) (xy 94.234 118.11))
-    (stroke (width 0) (type default))
-  )
-  (wire (pts (xy 90.805 56.134) (xy 90.805 57.658))
-    (stroke (width 0) (type default))
-  )
-  (wire (pts (xy 64.262 128.778) (xy 64.262 136.271))
-    (stroke (width 0) (type default))
-  )
-  (wire (pts (xy 85.09 65.151) (xy 114.427 65.151))
-    (stroke (width 0) (type default))
-  )
-  (wire (pts (xy 49.657 107.315) (xy 48.133 107.315))
-    (stroke (width 0) (type default))
-  )
-  (wire (pts (xy 45.593 117.475) (xy 45.593 120.65))
-    (stroke (width 0) (type default))
-  )
   (wire (pts (xy 41.148 120.65) (xy 45.593 120.65))
     (stroke (width 0) (type default))
   )
+  (wire (pts (xy 64.262 125.73) (xy 64.262 128.778))
+    (stroke (width 0) (type default))
+  )
   (wire (pts (xy 48.133 107.315) (xy 48.133 114.935))
     (stroke (width 0) (type default))
@@
   )
   (wire (pts (xy 66.802 133.858) (xy 69.342 133.858))
-    (stroke (width 0) (type default))
-  )
-  (wire (pts (xy 64.262 125.73) (xy 64.262 128.778))
     (stroke (width 0) (type default))
   )
@@
       (effects (font (size 0.77 0.77)) (justify left))
     )
-    (property "Footprint" "" (at 69.342 130.048 0)
+    (property "Footprint" "Capacitor_THT:CP_Axial_L10.0mm_D6.0mm_P15.00mm_Horizontal" (at 69.342 130.048 0)
       (effects (font (size 1.27 1.27)) hide)
     )
@@
       (effects (font (size 0.77 0.77)) (justify right))
     )
-    (property "Footprint" "" (at 82.55 65.151 0)
+    (property "Footprint" "Resistor_THT:R_Axial_DIN0309_L9.0mm_D3.2mm_P5.08mm_Vertical" (at 82.55 65.151 0)
       (effects (font (size 1.27 1.27)) hide)
     )
@@
       (effects (font (size 0.77 0.77)))
     )
-    (property "Footprint" "" (at 90.805 53.594 0)
+    (property "Footprint" "Resistor_THT:R_Axial_DIN0309_L9.0mm_D3.2mm_P5.08mm_Vertical" (at 90.805 53.594 0)
       (effects (font (size 1.27 1.27)) hide)
     )
@@
       (effects (font (size 0.77 0.77)) (justify left))
     )
-    (property "Footprint" "" (at 79.375 88.392 0)
+    (property "Footprint" "Capacitor_THT:CP_Axial_L10.0mm_D6.0mm_P15.00mm_Horizontal" (at 79.375 88.392 0)
       (effects (font (size 1.27 1.27)) hide)
     )
@@
       (effects (font (size 0.77 0.77)) (justify right))
     )
-    (property "Footprint" "" (at 45.593 114.935 0)
+    (property "Footprint" "Resistor_THT:R_Axial_DIN0309_L9.0mm_D3.2mm_P5.08mm_Vertical" (at 45.593 114.935 0)
       (effects (font (size 1.27 1.27)) hide)
     )
@@
       (effects (font (size 0.77 0.77)))
     )
-    (property "Footprint" "" (at 134.366 60.452 0)
+    (property "Footprint" "Resistor_THT:R_Axial_DIN0309_L9.0mm_D3.2mm_P5.08mm_Vertical" (at 134.366 60.452 0)
       (effects (font (size 1.27 1.27)) hide)
     )
@@
       (effects (font (size 0.77 0.77)) (justify right))
     )
-    (property "Footprint" "" (at 118.618 76.2 90)
+    (property "Footprint" "LED_THT:LED_D3.0mm" (at 118.618 76.2 90)
       (effects (font (size 1.27 1.27)) hide)
     )
@@
       (effects (font (size 0.77 0.77)))
     )
-    (property "Footprint" "" (at 122.809 71.501 0)
+    (property "Footprint" "Resistor_THT:R_Axial_DIN0309_L9.0mm_D3.2mm_P5.08mm_Vertical" (at 122.809 71.501 0)
       (effects (font (size 1.27 1.27)) hide)
     )
@@
       (effects (font (size 0.9 0.9)))
     )
-    (property "Footprint" "" (at 69.342 115.57 0)
+    (property "Footprint" "Package_DIP:DIP-8_W7.62mm_Socket" (at 69.342 115.57 0)
       (effects (font (size 1.27 1.27)) hide)
     )
@@
       (effects (font (size 0.7 0.7)))
     )
-    (property "Footprint" "" (at 52.197 107.315 0)
+    (property "Footprint" "Capacitor_THT:CP_Axial_L10.0mm_D6.0mm_P15.00mm_Horizontal" (at 52.197 107.315 0)
       (effects (font (size 1.27 1.27)) hide)
     )
@@
       (effects (font (size 0.77 0.77)) (justify left))
     )
-    (property "Footprint" "" (at 80.899 118.11 0)
-      (effects (font (size 1.27 1.27)) hide)
-    )
+    (property "Footprint" "Capacitor_THT:CP_Axial_L10.0mm_D6.0mm_P15.00mm_Horizontal" (at 80.899 118.11 0)
+      (effects (font (size 1.27 1.27)) hide)
+    )

Commit message: KiCAD schema bijgewerkt
Parts:
- added D2: Pwr LED, LED_THT:LED_D3.0mm, symbol Device:LED_Small
- added J2: NCJ6FA-H_Gitaar, Connector_Audio:Jack_XLR-6.35mm_Neutrik_NCJ6FA-H_Horizontal, symbol Connector_Audio:NCJ6FA-H
Connections:
- net +9V: now also D2.2 (A)
- net GND: now also D2.1 (K), J2.S
- net Signaal IN renamed Gitaar_IN
- net Gitaar_IN: now also J2.T
Other:
- moved on the sheet: C1, C2, C3, J1, RV1, U2

Commit message: KiCAD schema bijgewerkt
Parts:
- removed J1: Geluid_UIT, symbol Connector_Audio:AudioPlug2
- added J1: NCJ6FA-H_Gitaar, Connector_Audio:Jack_XLR-6.35mm_Neutrik_NCJ6FA-H_Horizontal, symbol Connector_Audio:NCJ6FA-H
- Q1: footprint (none) -> Package_TO_SOT_THT:TO-92L
Connections:
- net GND: now also J1.S
- net at C3.2: now also J1.R, J1.T
Changed lines of the file:
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@@
   (junction (at 118.618 71.501) (diameter 0) (color 0 0 0 0)
+  )
+  (junction (at 92.202 127.127) (diameter 0) (color 0 0 0 0)
   )
   (junction (at 50.165 118.999) (diameter 0) (color 0 0 0 0)
@@
     (stroke (width 0) (type default))
   )
+  (wire (pts (xy 92.202 127.127) (xy 92.202 129.667))
+    (stroke (width 0) (type default))
+  )
   (wire (pts (xy 79.375 93.091) (xy 97.282 93.091))
     (stroke (width 0) (type default))
@@
     (stroke (width 0) (type default))
   )
+  (wire (pts (xy 92.202 129.667) (xy 95.377 129.667))
+    (stroke (width 0) (type default))
+  )
   (polyline (pts (xy 22.225 153.543) (xy 136.017 153.543))
     (stroke (width 0) (type default))
@@
     (stroke (width 0) (type default))
   )
-  (wire (pts (xy 88.011 127.127) (xy 98.806 127.127))
+  (wire (pts (xy 88.011 127.127) (xy 92.202 127.127))
     (stroke (width 0) (type default))
   )
@@
     (stroke (width 0) (type default))
   )
+  (wire (pts (xy 91.694 124.587) (xy 91.694 117.475))
+    (stroke (width 0) (type default))
+  )
   (wire (pts (xy 97.282 66.421) (xy 97.282 57.658))
     (stroke (width 0) (type default))
@@
     (stroke (width 0) (type default))
   )
+  (wire (pts (xy 95.377 124.587) (xy 91.694 124.587))
+    (stroke (width 0) (type default))
+  )
   (wire (pts (xy 61.849 124.587) (xy 61.849 116.332))
     (stroke (width 0) (type default))
@@
     (stroke (width 0) (type default))
   )
-  (wire (pts (xy 96.901 132.207) (xy 96.901 135.636))
-    (stroke (width 0) (type default))
-  )
   (wire (pts (xy 134.366 56.261) (xy 134.366 57.912))
     (stroke (width 0) (type default))
@@
     (stroke (width 0) (type default))
   )
+  (wire (pts (xy 92.202 127.127) (xy 95.377 127.127))
+    (stroke (width 0) (type default))
+  )
   (wire (pts (xy 79.375 71.501) (xy 79.375 83.439))
-    (stroke (width 0) (type default))
-  )
-  (wire (pts (xy 98.806 132.207) (xy 96.901 132.207))
     (stroke (width 0) (type default))
   )
@@
     )
   )
+  (symbol (lib_id "Connector_Audio:NCJ6FA-H") (at 100.457 127.127 0) (mirror y) (unit 2)
+    (in_bom yes) (on_board yes) (dnp no)
+    (property "Reference" "J1" (at 102.362 120.015 0)
+      (effects (font (size 1.27 1.27)))
+    )
+    (property "Value" "NCJ6FA-H_Gitaar" (at 101.727 122.047 0)
+      (effects (font (size 0.6 0.6)))
+    )
+    (property "Footprint" "Connector_Audio:Jack_XLR-6.35mm_Neutrik_NCJ6FA-H_Horizontal" (at 100.457 127.127 0)
+      (effects (font (size 1.27 1.27)) hide)
+    )
+    (property "Datasheet" "https://www.neutrik.com/en/product/ncj6fa-h" (at 100.457 127.127 0)
+      (effects (font (size 1.27 1.27)) hide)
+    )
+    (pin "1")
+    (pin "2")
+    (pin "3")
+    (pin "G")
+    (pin "R")
+    (pin "S")
+    (pin "T")
+    (instances
+      (project "555-gitaar-pedal"
+        (path "/a176e3ad-e522-4300-abee-2d729589d26e"
+          (reference "J1") (unit 2)
+        )
+      )
+    )
+  )
   (symbol (lib_id "Device:R_Potentiometer_Small") (at 50.165 123.952 0) (unit 1)
     (in_bom yes) (on_board yes) (dnp no)
@@
         (path "/a176e3ad-e522-4300-abee-2d729589d26e"
           (reference "R1") (unit 1)
-        )
-      )
-    )
-  )
-  (symbol (lib_id "Connector_Audio:AudioPlug2") (at 114.046 129.667 180) (unit 1)
-    (in_bom yes) (on_board yes) (dnp no)
-    (property "Reference" "J1" (at 127.762 128.397 0)
-      (effects (font (size 1.27 1.27)) (justify right))
-    )
-    (property "Value" "Geluid_UIT" (at 106.68 127.254 0)
-      (effects (font (size 1.27 1.27)) (justify right))
-    )
-    (property "Footprint" "" (at 105.156 128.397 0)
-      (effects (font (size 1.27 1.27)) hide)
-    )
-    (property "Datasheet" "~" (at 105.156 128.397 0)
-      (effects (font (size 1.27 1.27)) hide)
-    )
-    (pin "S")
-    (pin "T")
-    (instances
-      (project "555-gitaar-pedal"
-        (path "/a176e3ad-e522-4300-abee-2d729589d26e"
-          (reference "J1") (unit 1)
         )
       )
@@
   (symbol (lib_id "Simulation_SPICE:PNP") (at 131.826 71.501 0) (unit 1)
     (in_bom yes) (on_board yes) (dnp no) (fields_autoplaced)
-    (property "Reference" "Q1" (at 136.8552 70.231 0)
-      (effects (font (size 1.27 1.27)) (justify left))
-    )
-    (property "Value" "BC547" (at 136.8552 72.771 0)
-      (effects (font (size 1.27 1.27)) (justify left))
-    )
-    (property "Footprint" "" (at 167.386 71.501 0)
+    (property "Reference" "Q1" (at 137.16 70.8659 0)
+      (effects (font (size 0.9 0.9)) (justify left))
+    )
+    (property "Value" "BC547" (at 137.16 72.771 0)
+      (effects (font (size 0.7 0.7)) (justify left))
+    )
+    (property "Footprint" "Package_TO_SOT_THT:TO-92L" (at 167.386 71.501 0)
       (effects (font (size 1.27 1.27)) hide)
     )
@@
     )
   )
-  (symbol (lib_id "power:GND") (at 96.901 135.636 0) (unit 1)
-    (in_bom yes) (on_board yes) (dnp no)
-    (property "Reference" "#PWR05" (at 96.901 141.986 0)
-      (effects (font (size 1.27 1.27)) hide)
-    )
-    (property "Value" "GND" (at 96.901 139.192 0)
+  (symbol (lib_id "power:GND") (at 91.694 117.475 90) (unit 1)
+    (in_bom yes) (on_board yes) (dnp no)
+    (property "Reference" "#PWR05" (at 98.044 117.475 0)
+      (effects (font (size 1.27 1.27)) hide)
+    )
+    (property "Value" "GND" (at 95.25 117.475 0)
       (effects (font (size 0.77 0.77)))
     )
-    (property "Footprint" "" (at 96.901 135.636 0)
-      (effects (font (size 1.27 1.27)) hide)
-    )
-    (property "Datasheet" "" (at 96.901 135.636 0)
-      (effects (font (size 1.27 1.27)) hide)
-    )
+    (property "Footprint" "" (at 91.694 117.475 0)
+      (effects (font (size 1.27 1.27)) hide)
+    )
+    (property "Datasheet" "" (at 91.694 117.475 0)
+      (effects (font (size 1.27 1.27)) hide)
+    )

Commit message: KiCAD schema bijgewerkt
Connections:
- net Gitaar_IN: now also J2.R
Changed lines of the file:
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@@
-    (stroke (width 0) (type default))
-  )
-  (wire (pts (xy 37.719 116.459) (xy 50.165 116.459))
     (stroke (width 0) (type default))
   )
@@
     (stroke (width 0) (type default))
   )
-  (wire (pts (xy 45.72 129.667) (xy 50.165 129.667))
+  (wire (pts (xy 68.834 134.747) (xy 68.834 137.795))
     (stroke (width 0) (type default))
   )
-  (wire (pts (xy 68.834 134.747) (xy 68.834 137.795))
+  (wire (pts (xy 45.72 129.667) (xy 50.165 129.667))
     (stroke (width 0) (type default))
   )
@@
     (stroke (width 0) (type default))
   )
+  (wire (pts (xy 37.592 116.459) (xy 50.165 116.459))
+    (stroke (width 0) (type default))
+  )
